File: RU First Prototype/STM 32 RU First Prototype.kicad_sch (KiCad schematic)
At the start: 81 parts, among them J1 Conn_01x02, J10 Conn_01x02_Pin, J11 Conn_01x02_Pin, J12 1776113-2, J2 USB_C_Receptacle, J3 Conn_01x02_Pin, J4 Conn_01x04, J5 Conn_01x02_Pin, J6 1776113-2, J7 1776113-2, J8 1776113-2, J9 Conn_01x02_Pin, Q1 SISA96DN-T1, Q2 SISA96DN-T1, Q3 SISA96DN-T1, Q4 SISA96DN-T1, SW1 SW_SPDT, U1 STM32F412RGTx, U2 AMS1117-3.3, U3 MS5611, U4 KX134-1211, U5 W25Q16JVSS, U6 TCAN330, U7 TCAN330, Y1 Crystal_8Mhz

Commit message: Started Laying traces
Parts:
- added C23, C24, C25, C26, C27, C28, C29, C30: 47pf, Capacitor_SMD:C_0201_0603Metric, symbol Device:C
- added C31, C32: 4.7n, Capacitor_SMD:C_0201_0603Metric, symbol Device:C
- added CR1, CR2, CR3, CR4: ESDCAN02-2BWY, ESDCAN02-2BWY:SOT323-3L_STM, symbol ESDCAN02-2BWY:ESDCAN02-2BWY
- added R24, R26, R27, R28: 60, Resistor_SMD:R_0201_0603Metric, symbol Device:R_Small_US
Connections:
- net ALT_CS: now also U1.59 (PB7); no longer U1.25 (PC5)
- net ALT_SCLK: now also U1.55 (PB3); no longer U1.21 (PA5)
- net Buzzer_G: now also U1.15 (PA1); no longer U1.22 (PA6)
- net CAN_H: now also J10.2 (Pin_2), J11.2 (Pin_2), C23.2, C26.2, CR1.2, CR3.2, R24.1; no longer J10.1 (Pin_1), J11.1 (Pin_1)
- net CAN_H2: now also C27.2, C30.2, CR2.2, CR4.2, R27.1
- net CAN_L2: now also C28.2, C29.2, CR2.1, CR4.1, R28.1
- net Drogue2: now also U1.51 (PC10); no longer U1.24 (PC4)
- net FLASH_IO0: now also U1.22 (PA6); no longer U1.40 (PC9)
- net FLASH_IO1: now also U1.23 (PA7); no longer U1.51 (PC10)
- net FLASH_IO2: now also U1.24 (PC4); no longer U1.39 (PC8)
- net FLASH_IO3: now also U1.25 (PC5); no longer U1.15 (PA1)
- net GND: now also C23.1, C24.1, C25.1, C26.1, C27.1, C28.1, C29.1, C30.1, C31.2, C32.2, CR1.3, CR2.3, CR3.3, CR4.3
- net KX_CS: now also U1.9 (PC1); no longer U1.20 (PA4)
- net KX_SCK: now also U1.38 (PC7); no longer U1.29 (PB10)
- net mLED: now also U1.40 (PC9); no longer U1.23 (PA7)
- new net: C32.1, R27.2, R28.2
- new net: C31.1, R24.2, R26.2
- new net CAN_L: C24.2, C25.2, CR1.1, CR3.1, J10.1 (Pin_1), J11.1 (Pin_1), R26.1, U6.6 (CANL)
- no-connect marks 3 -> 21
Other:
- moved on the sheet: J10, J11, J3, J9, R18, R19, R20

Commit message: Added some more traces
Parts:
- C1, C10, C11, C12, C13, C14, C15, C16, C17, C18, C19, C2, C20, C21, C22, C23, C24, C25, C26, C27, C28, C29, C3, C30, C31, C32, C4, C5, C6, C7, C8, C9: footprint Capacitor_SMD:C_0201_0603Metric -> Capacitor_SMD:C_0603_1608Metric
- R1, R10, R11, R12, R13, R14, R15, R16, R17, R18, R19, R2, R20, R21, R22, R23, R24, R25, R26, R27, R28, R3, R4, R5, R6, R7, R8, R9: footprint Resistor_SMD:R_0201_0603Metric -> Resistor_SMD:R_0603_1608Metric

Commit message: Changing XT30 connectors left
Connections:
- net Drogue: now also U1.39 (PC8); no longer U1.43 (PA10)
- net Drogue2: now also U1.40 (PC9); no longer U1.51 (PC10)
- net KX_SCK: now also U1.36 (PB15); no longer U1.38 (PC7)
- net PB15: now also U1.38 (PC7); no longer U1.36 (PB15)
- net mLED: now also U1.16 (PA2); no longer U1.40 (PC9)
Changed lines of the file:
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@@
 	)
 	(no_connect
-		(at 124.46 106.68)
+		(at 124.46 119.38)
 	)
 	(no_connect
-		(at 124.46 119.38)
+		(at 165.1 88.9)
 	)
 	(no_connect
@@
 	)
 	(no_connect
-		(at 165.1 68.58)
+		(at 124.46 86.36)
 	)
 	(no_connect
-		(at 124.46 86.36)
+		(at 124.46 111.76)
 	)
 	(no_connect
@@
 	)
 	(label "KX_SCK"
-		(at 124.46 104.14 180)
+		(at 165.1 142.24 0)
 		(effects
 			(font
 				(size 1.27 1.27)
 			)
-			(justify right bottom)
+			(justify left bottom)
 		)
 	)
@@
 	)
 	(label "PB15"
-		(at 165.1 142.24 0)
+		(at 124.46 104.14 180)
 		(effects
 			(font
 				(size 1.27 1.27)
 			)
-			(justify left bottom)
+			(justify right bottom)
 		)
 	)
@@
 	)
 	(label "mLED"
-		(at 124.46 109.22 180)
+		(at 165.1 68.58 0)
 		(effects
 			(font
 				(size 1.27 1.27)
 			)
-			(justify right bottom)
+			(justify left bottom)
 		)
 	)
@@
 	)
 	(label "Drogue2"
-		(at 124.46 111.76 180)
+		(at 124.46 109.22 180)
 		(effects
 			(font
@@
 	)
 	(label "Drogue"
-		(at 165.1 88.9 0)
+		(at 124.46 106.68 180)
 		(effects
 			(font
@@
 				(thickness 0.1588)
 			)
-			(justify left bottom)
+			(justify right bottom)
 		)
 	)

Commit message: Update
Parts:
- J1: footprint Connector_AMASS:AMASS_XT30PW-F_1x02_P2.50mm_Horizontal -> Connector_AMASS:AMASS_XT30U-M_1x02_P5.0mm_Vertical
- J10, J11, J3, J5, J9: footprint Connector_AMASS:AMASS_XT30PW-M_1x02_P2.50mm_Horizontal -> Connector_AMASS:AMASS_XT30U-M_1x02_P5.0mm_Vertical
Connections:
- net PC6: now also R22.2, R23.1; no longer R19.2, R20.1
- removed net PB15: R22.2, R23.1, U1.38 (PC7)
- new net PC7: R19.2, R20.1, U1.38 (PC7)
Changed lines of the file:
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@@
 		)
 	)
-	(label "PC6"
-		(at 254 143.51 180)
-		(effects
-			(font
-				(size 1.27 1.27)
-			)
-			(justify right bottom)
-		)
-	)
 	(label "CAN_H"
 		(at 114.3 177.8 90)
@@
 		)
 	)
+	(label "PC7"
+		(at 254 143.51 180)
+		(effects
+			(font
+				(size 1.27 1.27)
+			)
+			(justify right bottom)
+		)
+	)
 	(label "OSC_IN"
 		(at 110.49 67.31 180)
@@
 		)
 	)
-	(label "PB15"
-		(at 124.46 104.14 180)
+	(label "PC6"
+		(at 124.46 101.6 180)
 		(effects
 			(font
@@
 		)
 	)
+	(label "PC6"
+		(at 279.4 143.51 0)
+		(effects
+			(font
+				(size 1.27 1.27)
+			)
+			(justify left bottom)
+		)
+	)
 	(label "GND"
 		(at 87.63 146.05 0)
@@
 		)
 	)
-	(label "PB15"
-		(at 279.4 143.51 0)
-		(effects
-			(font
-				(size 1.27 1.27)
-			)
-			(justify left bottom)
-		)
-	)
 	(label "GND"
 		(at 270.51 151.13 270)
@@
 		)
 	)
-	(label "PC6"
-		(at 124.46 101.6 180)
+	(label "PC7"
+		(at 124.46 104.14 180)
 		(effects
 			(font
@@
 			)
 		)
-		(property "Footprint" "Connector_AMASS:AMASS_XT30PW-M_1x02_P2.50mm_Horizontal"
+		(property "Footprint" "Connector_AMASS:AMASS_XT30U-M_1x02_P5.0mm_Vertical"
 			(at 116.84 196.85 0)
 			(effects
@@
 			)
 		)
-		(property "Footprint" "Connector_AMASS:AMASS_XT30PW-M_1x02_P2.50mm_Horizontal"
+		(property "Footprint" "Connector_AMASS:AMASS_XT30U-M_1x02_P5.0mm_Vertical"
 			(at 189.23 170.18 0)
 			(effects
@@
 			)
 		)
-		(property "Footprint" "Connector_AMASS:AMASS_XT30PW-F_1x02_P2.50mm_Horizontal"
+		(property "Footprint" "Connector_AMASS:AMASS_XT30U-M_1x02_P5.0mm_Vertical"
 			(at 69.85 20.32 0)
 			(effects
@@
 			)
 		)
-		(property "Footprint" "Connector_AMASS:AMASS_XT30PW-M_1x02_P2.50mm_Horizontal"
+		(property "Footprint" "Connector_AMASS:AMASS_XT30U-M_1x02_P5.0mm_Vertical"
 			(at 172.72 152.4 0)
 			(effects
@@
 			)
 		)
-		(property "Footprint" "Connector_AMASS:AMASS_XT30PW-M_1x02_P2.50mm_Horizontal"
+		(property "Footprint" "Connector_AMASS:AMASS_XT30U-M_1x02_P5.0mm_Vertical"
 			(at 93.98 180.34 0)
 			(effects
@@
 			)
 		)
-		(property "Footprint" "Connector_AMASS:AMASS_XT30PW-M_1x02_P2.50mm_Horizontal"
+		(property "Footprint" "Connector_AMASS:AMASS_XT30U-M_1x02_P5.0mm_Vertical"
 			(at 271.78 53.34 0)
 			(effects

Commit message: Compactness ++
Parts:
- removed J6, J8: 1776113-2, 1776113-2:TE_1776113-2, symbol 1776113-2:1776113-2
- removed Q2, Q4: SISA96DN-T1, SISA96DN-T1:SIS862DNT1GE3, symbol SISA96DN-T1-GE3:SISA96DN-T1-GE3
- removed R12, R16: 10k, Resistor_SMD:R_0603_1608Metric, symbol Device:R_Small_US
- removed R13, R17: 100, Resistor_SMD:R_0603_1608Metric, symbol Device:R_Small_US
Connections:
- net V_MAIN: no longer Q1.10 (D_6), Q1.11 (D_7), Q1.5 (D_1), Q1.6 (D_2), Q1.7 (D_3), Q1.8 (D_4), Q1.9 (D_5)
- net Drogue2: no longer names the net of U1.40 (PC9)
- net Main2: no longer names the net of U1.42 (PA9)
- new net: Q1.10 (D_6), Q1.11 (D_7), Q1.5 (D_1), Q1.6 (D_2), Q1.7 (D_3), Q1.8 (D_4), Q1.9 (D_5)
- no-connect marks 21 -> 23
Other:
- moved on the sheet: Q1, R10, R11
