File: RU First Prototype/STM 32 RU First Prototype.kicad_sch (KiCad schematic)
At the start: 91 parts, among them J1 Conn_01x02, J10 Conn_01x02_Pin, J11 Conn_01x02_Pin, J12 1776113-2, J2 USB_C_Receptacle, J3 Conn_01x02_Pin, J4 Conn_01x04, J5 Conn_01x02_Pin, J7 1776113-2, J9 Conn_01x02_Pin, Q1 SISA96DN-T1, Q3 SISA96DN-T1, SW1 SW_SPDT, U1 STM32F412RGTx, U2 AMS1117-3.3, U3 MS5611, U4 KX134-1211, U5 W25Q16JVSS, U6 TCAN330, U7 TCAN330, Y1 Crystal_8Mhz

Commit message: Fixed schematic and some routing, flash routing left
Connections:
- net +3V3: no longer U1.1 (VBAT)
- net ALT_CS: now also U1.20 (PA4); no longer U1.9 (PC1)
- net ALT_SCLK: now also U1.21 (PA5); no longer U1.36 (PB15)
- net ALT_SDI: now also U1.22 (PA6); no longer U1.11 (PC3)
- net ALT_SDO: now also U1.23 (PA7); no longer U1.10 (PC2)
- net Buzzer_G: now also U1.14 (PA0); no longer U1.15 (PA1)
- net CAN_RX2: now also U1.33 (PB12); no longer U1.35 (PB14)
- net Drogue: now also U1.42 (PA9); no longer U1.39 (PC8)
- net FLASH_IO0: now also U1.40 (PC9); no longer U1.22 (PA6)
- net FLASH_IO1: now also U1.51 (PC10); no longer U1.23 (PA7)
- net FLASH_IO2: now also U1.39 (PC8); no longer U1.24 (PC4)
- net FLASH_IO3: now also U1.15 (PA1); no longer U1.25 (PC5)
- net KX_SDI: now also U1.52 (PC11); no longer U1.57 (PB5)
- net KX_SDO: now also U1.53 (PC12); no longer U1.56 (PB4)
- no-connect marks 23 -> 25
Changed lines of the file:
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@@
 	)
 	(junction
-		(at 144.78 151.13)
-		(diameter 0)
-		(color 0 0 0 0)
-	)
-	(junction
 		(at 109.22 53.34)
 		(diameter 0)
@@
 	)
 	(junction
+		(at 144.78 151.13)
+		(diameter 0)
+		(color 0 0 0 0)
+	)
+	(junction
 		(at 157.48 168.91)
 		(diameter 0)
@@
 	)
 	(junction
-		(at 144.78 53.34)
-		(diameter 0)
-		(color 0 0 0 0)
-	)
-	(junction
 		(at 209.55 82.55)
 		(diameter 0)
@@
 	)
 	(no_connect
-		(at 165.1 134.62)
-	)
-	(no_connect
 		(at 15.24 166.37)
 	)
 	(no_connect
-		(at 165.1 86.36)
-	)
-	(no_connect
 		(at 124.46 121.92)
 	)
 	(no_connect
-		(at 124.46 109.22)
+		(at 124.46 99.06)
 	)
 	(no_connect
@@
 	)
 	(no_connect
-		(at 124.46 81.28)
+		(at 165.1 139.7)
 	)
 	(no_connect
-		(at 165.1 63.5)
+		(at 124.46 81.28)
 	)
 	(no_connect
-		(at 124.46 116.84)
+		(at 124.46 88.9)
 	)
 	(no_connect
-		(at 165.1 73.66)
+		(at 165.1 119.38)
 	)
 	(no_connect
-		(at 124.46 114.3)
+		(at 124.46 93.98)
 	)
 	(no_connect
@@
 	)
 	(no_connect
-		(at 124.46 86.36)
+		(at 125.73 93.98)
 	)
 	(no_connect
-		(at 124.46 111.76)
+		(at 124.46 86.36)
 	)
 	(no_connect
@@
 	)
 	(no_connect
-		(at 165.1 76.2)
+		(at 124.46 96.52)
+	)
+	(no_connect
+		(at 189.23 77.47)
+	)
+	(no_connect
+		(at 124.46 91.44)
+	)
+	(no_connect
+		(at 165.1 142.24)
 	)
 	(no_connect
 		(at 165.1 101.6)
 	)
+	(no_connect
+		(at 165.1 116.84)
+	)
 	(wire
 		(pts
@@
 	(wire
 		(pts
+			(xy 144.78 151.13) (xy 147.32 151.13)
+		)
+		(stroke
+			(width 0)
+			(type default)
+		)
+	)
+	(wire
+		(pts
 			(xy 58.42 177.8) (xy 55.88 177.8)
 		)
@@
 	(wire
 		(pts
-			(xy 139.7 53.34) (xy 142.24 53.34)
-		)
-		(stroke
-			(width 0)
-			(type default)
-		)
-	)
-	(wire
-		(pts
 			(xy 177.8 143.51) (xy 177.8 144.78)
 		)
@@
 	(wire
 		(pts
-			(xy 118.11 91.44) (xy 124.46 91.44)
-		)
-		(stroke
-			(width 0)
-			(type default)
-		)
-	)
-	(wire
-		(pts
 			(xy 125.73 191.77) (xy 124.46 191.77)
 		)
@@
 	(wire
 		(pts
-			(xy 144.78 151.13) (xy 147.32 151.13)
-		)
-		(stroke
-			(width 0)
-			(type default)
-		)
-	)
-	(wire
-		(pts
 			(xy 64.77 170.18) (xy 67.31 170.18)
 		)
@@
 	)
 	(label "FLASH_IO0"
-		(at 165.1 78.74 0)
+		(at 124.46 109.22 180)
 		(effects
 			(font
 				(size 1.27 1.27)
 			)
-			(justify left bottom)
+			(justify right bottom)
 		)
 	)
@@
 	)
 	(label "FLASH_IO1"
-		(at 165.1 81.28 0)
+		(at 124.46 111.76 180)
 		(effects
 			(font
 				(size 1.27 1.27)
 			)
-			(justify left bottom)
+			(justify right bottom)
 		)
 	)
@@
 	)
 	(label "FLASH_IO3"
-		(at 124.46 99.06 180)
+		(at 165.1 66.04 0)
 		(effects
 			(font
 				(size 1.27 1.27)
 			)
-			(justify right bottom)
+			(justify left bottom)
 		)
 	)
@@
 	)
 	(label "ALT_SCLK"
-		(at 165.1 142.24 0)
+		(at 165.1 76.2 0)
 		(effects
 			(font
@@
 	)
 	(label "ALT_CS"
-		(at 124.46 88.9 180)
+		(at 165.1 73.66 0)
 		(effects
 			(font
 				(size 1.27 1.27)
 			)
-			(justify right bottom)
+			(justify left bottom)
 		)
 	)
@@
 	)
 	(label "KX_SDO"
-		(at 165.1 116.84 0)
+		(at 124.46 116.84 180)
 		(effects
 			(font
 				(size 1.27 1.27)
 			)
-			(justify left bottom)
+			(justify right bottom)
 		)
 	)
 	(label "FLASH_IO2"
-		(at 124.46 96.52 180)
+		(at 124.46 106.68 180)
 		(effects
 			(font
@@
 	)
 	(label "CAN_RX2"
-		(at 165.1 139.7 0)
+		(at 165.1 134.62 0)
 		(effects
 			(font
@@
 	)
 	(label "ALT_SDO"
-		(at 118.11 91.44 180)
+		(at 165.1 81.28 0)
 		(effects
 			(font
 				(size 1.27 1.27)
 			)
-			(justify right bottom)
+			(justify left bottom)
 		)
 	)
@@
 	)
 	(label "KX_SDI"
-		(at 165.1 119.38 0)
+		(at 124.46 114.3 180)
 		(effects
 			(font
 				(size 1.27 1.27)
 			)
-			(justify left bottom)
+			(justify right bottom)
 		)
 	)
@@
 	)
 	(label "ALT_SDI"
-		(at 124.46 93.98 180)
+		(at 165.1 78.74 0)
 		(effects
 			(font
 				(size 1.27 1.27)
 			)
-			(justify right bottom)
+			(justify left bottom)
 		)
 	)
@@
 	)
 	(label "Buzzer_G"
-		(at 165.1 66.04 0)
+		(at 165.1 63.5 0)
 		(effects
 			(font
@@
 	)
 	(label "Drogue"
-		(at 124.46 106.68 180)
+		(at 165.1 86.36 0)
 		(effects
 			(font
@@
 				(thickness 0.1588)
 			)
-			(justify right bottom)
+			(justify left bottom)
 		)
 	)

Commit message: Added flash chip and CAN bus 2 connections
Connections:
- net +3V3: now also U1.1 (VBAT)
Changed lines of the file:
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@@
+	(wire
+		(pts
+			(xy 139.7 53.34) (xy 142.24 53.34)
+		)
+		(stroke
+			(width 0)
+			(type default)
+		)
+	)
 	(wire
 		(pts

Commit message: Fixed SDO-SDI, Added Battery monitoring, and ADC inputs
Parts:
- added R29, R30: 10k, Resistor_SMD:R_0603_1608Metric, symbol Device:R_Small_US
- added R31: 13k, Resistor_SMD:R_0603_1608Metric, symbol Device:R_Small_US
Connections:
- net ALT_SDI: now also U1.23 (PA7); no longer U1.22 (PA6)
- net ALT_SDO: now also U1.22 (PA6); no longer U1.23 (PA7)
- net GND: now also R31.2
- net KX_SDI: now also U1.53 (PC12); no longer U1.52 (PC11)
- net KX_SDO: now also U1.52 (PC11); no longer U1.53 (PC12)
- net V_2S: now also R29.1
- net Main_Sense: now reaches U1.24 (PC4)
- net Main_Sense: now also R19.2, R20.1
- net Drogue_Sense: now reaches U1.26 (PB0)
- net Drogue_Sense: now also R22.2, R23.1
- net Bat_Sense: now reaches U1.9 (PC1)
- net Bat_Sense: now also R30.2, R31.1
- removed net PC6: R22.2, R23.1, U1.37 (PC6)
- removed net PC7: R19.2, R20.1, U1.38 (PC7)
- new net: R29.2, R30.1
- no-connect marks 25 -> 24
