File: RU First Prototype/_restore_backup_2026-09-07T07-34-59-787/STM 32 RU First Prototype.kicad_pcb (KiCad board)
At the start: 4 copper layers, 45 x 81.5 mm, 98 parts, among them J1 Conn_01x02, J10 Conn_01x02_Pin, J11 Conn_01x02_Pin, J12 1776113-2, J2 USB_C_Receptacle, J3 Conn_01x02_Pin, J4 Conn_01x04, J5 Conn_01x02_Pin, J7 1776113-2, J9 Conn_01x02_Pin, Q1 SISA96DN-T1, Q3 SISA96DN-T1, SW1 SW_SPDT, U1 STM32F412RGTx, U2 AMS1117-3.3, U3 MS5611, U4 KX134-1211, U5 W25Q16JVSS, U6 TCAN330, U7 TCAN330, Y1 Crystal_8Mhz

Commit message: made some more changes
Other:
- board text added: "RU"
- board text removed: "RECOVERY UNIT"
