File: RU First Prototype/_restore_backup_2026-09-07T07-34-59-787/STM 32 RU First Prototype.kicad_sch (KiCad schematic)
At the start: 91 parts, among them J1 Conn_01x02, J10 Conn_01x02_Pin, J11 Conn_01x02_Pin, J12 1776113-2, J2 USB_C_Receptacle, J3 Conn_01x02_Pin, J4 Conn_01x04, J5 Conn_01x02_Pin, J7 1776113-2, J9 Conn_01x02_Pin, Q1 SISA96DN-T1, Q3 SISA96DN-T1, SW1 SW_SPDT, U1 STM32F412RGTx, U2 AMS1117-3.3, U3 MS5611, U4 KX134-1211, U5 W25Q16JVSS, U6 TCAN330, U7 TCAN330, Y1 Crystal_8Mhz

Commit message: made some more changes
Parts:
- J10, J11, J3, J9: footprint Connector_PinHeader_2.54mm:PinHeader_1x02_P2.54mm_Vertical -> Connector_AMASS:AMASS_XT30U-M_1x02_P5.0mm_Vertical
- Q5: value (none) -> ~
