File: RU First Prototype/_restore_backup_2026-09-07T18-52-53-997/STM 32 RU First Prototype.kicad_sch (KiCad schematic)
At the start: 91 parts, among them J1 Conn_01x02, J10 Conn_01x02_Pin, J11 Conn_01x02_Pin, J12 1776113-2, J2 USB_C_Receptacle, J3 Conn_01x02_Pin, J4 Conn_01x04, J5 Conn_01x02_Pin, J7 1776113-2, J9 Conn_01x02_Pin, Q1 SISA96DN-T1, Q3 SISA96DN-T1, SW1 SW_SPDT, U1 STM32F412RGTx, U2 AMS1117-3.3, U3 MS5611, U4 KX134-1211, U5 W25Q16JVSS, U6 TCAN330, U7 TCAN330, Y1 Crystal_8Mhz

Commit message: Final touch done from my side
Connections:
- net ALT_CS: now also U1.59 (PB7); no longer U1.9 (PC1)
- net ALT_SCLK: now also U1.55 (PB3); no longer U1.36 (PB15)
- net ALT_SDI: now also U1.57 (PB5); no longer U1.11 (PC3)
- net ALT_SDO: now also U1.56 (PB4); no longer U1.10 (PC2)
- net KX_CS: now also U1.9 (PC1); no longer U1.59 (PB7)
- net KX_SCK: now also U1.36 (PB15); no longer U1.55 (PB3)
- net KX_SDI: now also U1.11 (PC3); no longer U1.57 (PB5)
- net KX_SDO: now also U1.10 (PC2); no longer U1.56 (PB4)
